File: battery-dc-dc-converter.sch (KiCad schematic (older format))
At the start: 22 parts, among them J1 Conn_01x02, J2 Conn_01x01, J3 Conn_01x01, U1 LMR16020

Commit message: Order v0.2
Parts:
- added C3: 220nF, Capacitor_SMD:C_0805_2012Metric, symbol Device:C
- C7: renamed from C12; value 470nF -> 220nF
- D1: LCSC C360444 -> C22452
- F1, F2: LCSC C182441 -> C140478
- R3: LCSC C39050 -> C25804
- R7: value 3R3 -> 3.3R; footprint Resistor_SMD:R_0805_2012Metric -> Resistor_SMD:R_0805_2012Metric_Pad1.20x1.40mm_HandSolder
- U1: LCSC (none) -> C190006
- renumbered C10 to C5, C11 to C6, C7 to C8
Connections:
- net GND: now also C3.2
- net VCC: now also C3.1
Changed lines of the file:
@@
 F 2 "Diode_SMD:D_SMA" H 6450 3700 50  0001 C CNN
 F 3 "~" H 6450 3700 50  0001 C CNN
-F 4 "C360444" H 6450 3700 50  0001 C CNN "LCSC"
+F 4 "C22452" H 6450 3700 50  0001 C CNN "LCSC"
 	1    6450 3700
 	1    0    0    -1
@@
 $EndComp
 $Comp
-L Device:C C7
+L Device:C C8
 U 1 1 5F47AD14
 P 7500 3950
-F 0 "C7" H 7615 3996 50  0000 L CNN
+F 0 "C8" H 7615 3996 50  0000 L CNN
 F 1 "1uF" H 7615 3905 50  0000 L CNN
 F 2 "Capacitor_SMD:C_0603_1608Metric" H 7538 3800 50  0001 C CNN
@@
 F 2 "Resistor_SMD:R_0603_1608Metric" V 7080 4150 50  0001 C CNN
 F 3 "~" H 7150 4150 50  0001 C CNN
-F 4 "C39050" H 7150 4150 50  0001 C CNN "LCSC"
+F 4 "C25804" H 7150 4150 50  0001 C CNN "LCSC"
 	1    7150 4150
 	1    0    0    -1
@@
 F 2 "Fuse:Fuse_1206_3216Metric_Pad1.42x1.75mm_HandSolder" V 1330 1000 50  0001 C CNN
 F 3 "~" H 1400 1000 50  0001 C CNN
-F 4 "C182441" H 1400 1000 50  0001 C CNN "LCSC"
+F 4 "C140478" H 1400 1000 50  0001 C CNN "LCSC"
 	1    1400 1000
 	0    1    1    0
@@
 F 2 "Fuse:Fuse_1206_3216Metric_Pad1.42x1.75mm_HandSolder" V 3280 1300 50  0001 C CNN
 F 3 "~" H 3350 1300 50  0001 C CNN
-F 4 "C182441" H 3350 1300 50  0001 C CNN "LCSC"
+F 4 "C140478" H 3350 1300 50  0001 C CNN "LCSC"
 	1    3350 1300
 	0    1    1    0
@@
 $EndComp
 Wire Wire Line
-	2850 3050 3750 3050
+	2850 3050 3250 3050
 $Comp
 L power:GND #PWR0114
@@
 P 5950 3450
 F 0 "R7" V 5743 3450 50  0000 C CNN
-F 1 "3R3" V 5834 3450 50  0000 C CNN
-F 2 "Resistor_SMD:R_0805_2012Metric" V 5880 3450 50  0001 C CNN
+F 1 "3.3R" V 5834 3450 50  0000 C CNN
+F 2 "Resistor_SMD:R_0805_2012Metric_Pad1.20x1.40mm_HandSolder" V 5880 3450 50  0001 C CNN
 F 3 "~" H 5950 3450 50  0001 C CNN
 F 4 "C24787" H 5950 3450 50  0001 C CNN "LCSC"
@@
 	5350 3950 7150 3950
 $Comp
-L Device:C C10
+L Device:C C5
 U 1 1 5F4F6FC9
 P 2150 3250
-F 0 "C10" H 2265 3296 50  0000 L CNN
+F 0 "C5" H 2265 3296 50  0000 L CNN
 F 1 "2.2uF" H 2150 3150 50  0000 L CNN
 F 2 "Capacitor_SMD:C_1210_3225Metric" H 2188 3100 50  0001 C CNN
@@
 $EndComp
 $Comp
-L Device:C C11
+L Device:C C6
 U 1 1 5F4F58E3
 P 2500 3250
-F 0 "C11" H 2615 3296 50  0000 L CNN
+F 0 "C6" H 2615 3296 50  0000 L CNN
 F 1 "2.2uF" H 2500 3150 50  0000 L CNN
 F 2 "Capacitor_SMD:C_1210_3225Metric" H 2538 3100 50  0001 C CNN
@@
 $EndComp
 $Comp
-L Device:C C12
+L Device:C C7
 U 1 1 5F4F514D
 P 2850 3250
-F 0 "C12" H 2965 3296 50  0000 L CNN
-F 1 "470nF" H 2850 3150 50  0000 L CNN
+F 0 "C7" H 2965 3296 50  0000 L CNN
+F 1 "220nF" H 2850 3150 50  0000 L CNN
 F 2 "Capacitor_SMD:C_0805_2012Metric" H 2888 3100 50  0001 C CNN
 F 3 "~" H 2850 3250 50  0001 C CNN
@@
 F 2 "Package_SO:HTSOP-8-1EP_3.9x4.9mm_P1.27mm_EP2.4x3.2mm" H 4900 3800 50  0001 C CNN
 F 3 "" H 4900 3800 50  0001 C CNN
+F 4 "C190006" H 4900 3800 50  0001 C CNN "LCSC"
 	1    4900 3800
 	1    0    0    -1
@@
 	1400 1100 1400 1150
 Connection ~ 1250 1100
+Wire Wire Line
+	3250 3400 3250 3450
+$Comp
+L Device:C C3
+U 1 1 616DB10B
+P 3250 3250
+F 0 "C3" H 3365 3296 50  0000 L CNN
+F 1 "220nF" H 3250 3150 50  0000 L CNN
+F 2 "Capacitor_SMD:C_0805_2012Metric" H 3288 3100 50  0001 C CNN
+F 3 "~" H 3250 3250 50  0001 C CNN
+F 4 "C513710" H 3250 3250 50  0001 C CNN "LCSC"
+	1    3250 3250
+	1    0    0    -1
+$EndComp
+Wire Wire Line
+	2850 3450 3250 3450
+Connection ~ 2850 3450
+Wire Wire Line
+	3250 3100 3250 3050
+Connection ~ 3250 3050
+Wire Wire Line
+	3250 3050 3750 3050
 $EndSCHEMATC
