File: battery-dc-dc-converter.sch (KiCad schematic (older format))
At the start: 23 parts, among them J1 Conn_01x02, J2 Conn_01x01, J3 Conn_01x01, U1 LMR16020

Commit message: Put power plug on same side
Parts:
- added C10, C11: 22uF, Capacitor_SMD:C_0805_2012Metric, symbol Device:C
- added C9: 2.2uF, Capacitor_SMD:C_1210_3225Metric, symbol Device:C
- R7: footprint Resistor_SMD:R_0805_2012Metric_Pad1.20x1.40mm_HandSolder -> Resistor_SMD:R_0805_2012Metric
- U1: LCSC C190006 -> C90665
Connections:
- net +12V: now also C10.1, C11.1
- net GND: now also C10.2, C11.2, C9.2
- net VCC: now also C9.1
Changed lines of the file:
@@
 F 0 "R7" V 5743 3450 50  0000 C CNN
 F 1 "3.3R" V 5834 3450 50  0000 C CNN
-F 2 "Resistor_SMD:R_0805_2012Metric_Pad1.20x1.40mm_HandSolder" V 5880 3450 50  0001 C CNN
+F 2 "Resistor_SMD:R_0805_2012Metric" V 5880 3450 50  0001 C CNN
 F 3 "~" H 5950 3450 50  0001 C CNN
 F 4 "C24787" H 5950 3450 50  0001 C CNN "LCSC"
@@
 F 2 "Package_SO:HTSOP-8-1EP_3.9x4.9mm_P1.27mm_EP2.4x3.2mm" H 4900 3800 50  0001 C CNN
 F 3 "" H 4900 3800 50  0001 C CNN
-F 4 "C190006" H 4900 3800 50  0001 C CNN "LCSC"
+F 4 "C90665" H 4900 3800 50  0001 C CNN "LCSC"
 	1    4900 3800
 	1    0    0    -1
@@
 Wire Wire Line
 	3250 3050 3750 3050
+$Comp
+L Device:C C9
+U 1 1 6181C331
+P 1800 3250
+F 0 "C9" H 1915 3296 50  0000 L CNN
+F 1 "2.2uF" H 1800 3150 50  0000 L CNN
+F 2 "Capacitor_SMD:C_1210_3225Metric" H 1838 3100 50  0001 C CNN
+F 3 "~" H 1800 3250 50  0001 C CNN
+F 4 "C106115" H 1800 3250 50  0001 C CNN "LCSC"
+	1    1800 3250
+	1    0    0    -1
+$EndComp
+Wire Wire Line
+	2150 3050 1800 3050
+Wire Wire Line
+	1800 3050 1800 3100
+Wire Wire Line
+	2150 3450 1800 3450
+Wire Wire Line
+	1800 3450 1800 3400
+$Comp
+L Device:C C10
+U 1 1 618243CA
+P 8750 3950
+F 0 "C10" H 8865 3996 50  0000 L CNN
+F 1 "22uF" H 8865 3905 50  0000 L CNN
+F 2 "Capacitor_SMD:C_0805_2012Metric" H 8788 3800 50  0001 C CNN
+F 3 "~" H 8750 3950 50  0001 C CNN
+F 4 "C45783" H 8750 3950 50  0001 C CNN "LCSC"
+	1    8750 3950
+	1    0    0    -1
+$EndComp
+$Comp
+L Device:C C11
+U 1 1 6182654C
+P 9200 3950
+F 0 "C11" H 9315 3996 50  0000 L CNN
+F 1 "22uF" H 9315 3905 50  0000 L CNN
+F 2 "Capacitor_SMD:C_0805_2012Metric" H 9238 3800 50  0001 C CNN
+F 3 "~" H 9200 3950 50  0001 C CNN
+F 4 "C45783" H 9200 3950 50  0001 C CNN "LCSC"
+	1    9200 3950
+	1    0    0    -1
+$EndComp
+Wire Wire Line
+	8300 4150 8750 4150
+Wire Wire Line
+	8750 4150 8750 4100
+Wire Wire Line
+	8750 4150 9200 4150
+Wire Wire Line
+	9200 4150 9200 4100
+Connection ~ 8750 4150
+Wire Wire Line
+	8750 3800 8750 3450
+Wire Wire Line
+	8750 3450 8300 3450
+Wire Wire Line
+	9200 3800 9200 3450
+Wire Wire Line
+	9200 3450 8750 3450
+Connection ~ 8750 3450
 $EndSCHEMATC
