File: battery-dc-dc-converter/battery-dc-dc-converter.kicad_pcb (KiCad board)
At the start: 4 copper layers, 42 x 33 mm, 30 parts, among them J1 Conn_01x02, J2 Conn_01x01, J3 Conn_01x01, U1 LMR16030P

Commit message: Tidy up
Parts:
- F1, F2: value 3A -> 4A
- moved REF** 0.81 mm to (131.4, 35.0)
- moved REF** 0.74 mm to (131.4, 69.0)
- moved REF** 0.58 mm to (107.0, 69.0)
- moved J2 0.25 mm to (110.7, 39.2)
Connections:
- net Net-(J1-Pin_2) renamed /VCC_Pre_Fuse
- net Net-(J2-Pin_1) renamed /12V_Fused
Other:
- board text added: "DC-DC Converter Input: 13-60V Output: 12V Max Output: 3A"
- board text removed: "DC-DC converter Vin: 13-60V Vout: 12V Max Out: 3A"
Changed lines of the file:
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@@
 	(net 5 "Net-(R5-Pad2)")
 	(net 6 "/SW")
-	(net 7 "Net-(J1-Pin_2)")
-	(net 8 "Net-(J2-Pin_1)")
+	(net 7 "/VCC_Pre_Fuse")
+	(net 8 "/12V_Fused")
 	(net 9 "Net-(U1-RT{slash}SYNC)")
 	(net 10 "/FB")
@@
 			)
 		)
-		(property "Value" "3A"
+		(property "Value" "4A"
 			(at 0 1.82 0)
 			(layer "F.Fab")
@@
 			)
 		)
-		(property "LCSC" "C140478"
+		(property "LCSC" "C136349"
 			(at 0 0 0)
 			(layer "F.Fab")
@@
 			(layers "F.Cu" "F.Paste" "F.Mask")
 			(roundrect_rratio 0.175439)
-			(net 8 "Net-(J2-Pin_1)")
+			(net 8 "/12V_Fused")
 			(pintype "passive")
 		)
@@
 	(footprint "battery-dc-dc-converter:hole-pad"
 		(layer "F.Cu")
-		(at 110.7 39.45)
+		(at 110.7 39.2)
 		(property "Reference" "J2"
 			(at 0 0.5 0)
@@
 			(remove_unused_layers no)
 			(roundrect_rratio 0.25)
-			(net 8 "Net-(J2-Pin_1)")
+			(net 8 "/12V_Fused")
 			(pinfunction "Pin_1")
 			(pintype "passive")
@@
 		(tags "resistor")
 		(property "Reference" "R3"
-			(at 0 -1.43 270)
+			(at 0 -1.43 -90)
 			(layer "F.SilkS")
 			(hide yes)
@@
 		(tags "capacitor")
 		(property "Reference" "C2"
-			(at -2.95 0 360)
+			(at -2.95 0 0)
 			(layer "F.SilkS")
 			(hide yes)
@@
 		)
 		(property "Value" "22uF"
-			(at 0 1.65 360)
+			(at 0 1.65 0)
 			(layer "F.Fab")
 			(effects
@@
 		)
 		(property "Footprint" "Capacitor_SMD:C_0805_2012Metric"
-			(at 0 0 360)
+			(at 0 0 0)
 			(layer "F.Fab")
 			(hide yes)
@@
 		)
 		(property "Datasheet" ""
-			(at 0 0 360)
+			(at 0 0 0)
 			(layer "F.Fab")
 			(hide yes)
@@
 		)
 		(property "Description" ""
-			(at 0 0 360)
+			(at 0 0 0)
 			(layer "F.Fab")
 			(hide yes)
@@
 		)
 		(fp_text user "${REFERENCE}"
-			(at 0 0 360)
+			(at 0 0 0)
 			(layer "F.Fab")
 			(effects
@@
 		(tags "capacitor")
 		(property "Reference" "C6"
-			(at -2.95 -0.05 360)
+			(at -2.95 -0.05 0)
 			(layer "F.SilkS")
 			(hide yes)
@@
 		)
 		(property "LCSC" "C55151"
-			(at 181.15 -64.25 360)
+			(at 181.15 -64.25 0)
 			(layer "F.Fab")
 			(hide yes)
@@
 		(tags "capacitor")
 		(property "Reference" "C5"
-			(at 1.45 -2.55 360)
+			(at 1.45 -2.55 0)
 			(layer "F.SilkS")
 			(hide yes)
@@
 		)
 		(property "LCSC" "C55151"
-			(at 62.25 190.65 360)
+			(at 62.25 190.65 0)
 			(layer "F.Fab")
 			(hide yes)
@@
 			(layers "*.Cu" "*.Mask")
 			(remove_unused_layers no)
-			(net 7 "Net-(J1-Pin_2)")
+			(net 7 "/VCC_Pre_Fuse")
 			(pinfunction "Pin_2")
 			(pintype "passive")
@@
 			)
 		)
-		(property "Value" "3A"
+		(property "Value" "4A"
 			(at 0 1.82 90)
 			(layer "F.Fab")
@@
 			)
 		)
-		(property "LCSC" "C140478"
+		(property "LCSC" "C136349"
 			(at 178.15 -61.25 0)
 			(layer "F.Fab")
@@
 			(layers "F.Cu" "F.Paste" "F.Mask")
 			(roundrect_rratio 0.175439)
-			(net 7 "Net-(J1-Pin_2)")
+			(net 7 "/VCC_Pre_Fuse")
 			(pintype "passive")
 		)
@@
 		(tags "resistor")
 		(property "Reference" "R5"
-			(at 0 -1.43 360)
+			(at 0 -1.43 0)
 			(layer "F.SilkS")
 			(hide yes)
@@
 		)
 		(property "Value" "33K"
-			(at 0 1.43 360)
+			(at 0 1.43 0)
 			(layer "F.Fab")
 			(effects
@@
 		)
 		(fp_text user "${REFERENCE}"
-			(at 0 0 360)
+			(at 0 0 0)
 			(layer "F.Fab")
 			(effects
@@
 		(tags "capacitor")
 		(property "Reference" "C11"
-			(at 0 1.8 360)
+			(at 0 1.8 0)
 			(layer "F.SilkS")
 			(hide yes)
@@
 		)
 		(property "Value" "22uF"
-			(at 0 1.65 360)
+			(at 0 1.65 0)
 			(layer "F.Fab")
 			(effects
@@
 		)
 		(property "Footprint" "Capacitor_SMD:C_0805_2012Metric"
-			(at 0 0 360)
+			(at 0 0 0)
 			(layer "F.Fab")
 			(hide yes)
@@
 		)
 		(property "Datasheet" ""
-			(at 0 0 360)
+			(at 0 0 0)
 			(layer "F.Fab")
 			(hide yes)
@@
 		)
 		(property "Description" ""
-			(at 0 0 360)
+			(at 0 0 0)
 			(layer "F.Fab")
 			(hide yes)
@@
 		)
 		(fp_text user "${REFERENCE}"
-			(at 0 0 360)
+			(at 0 0 0)
 			(layer "F.Fab")
 			(effects
@@
 		(tags "resistor")
 		(property "Reference" "R2"
-			(at 0 -1.43 270)
+			(at 0 -1.43 -90)
 			(layer "F.SilkS")
 			(hide yes)
@@
 	(footprint "PCM_kikit:Tab"
 		(layer "F.Cu")
-		(at 131.4 69.74 90)
+		(at 131.4 69 90)
 		(descr "A symbol representing annotation for tab placement")
 		(property "Reference" "REF**"
@@
 		)
 		(fp_text user "KIKIT: width: 4mm"
-			(at -5.5 0 360)
+			(at -5.5 0 0)
 			(layer "Dwgs.User")
 			(effects
@@
 	(footprint "PCM_kikit:Tab"
 		(layer "F.Cu")
-		(at 107 69.58 90)
+		(at 107 69 90)
 		(descr "A symbol representing annotation for tab placement")
 		(property "Reference" "REF**"
@@
 		)
 		(fp_text user "KIKIT: width: 4mm"
-			(at -5.5 0 360)
+			(at -5.5 0 0)
 			(layer "Dwgs.User")
 			(effects
@@
 		)
 		(fp_text user "KIKIT: width: 4mm"
-			(at -5.5 0 360)
+			(at -5.5 0 0)
 			(layer "Dwgs.User")
 			(effects
@@
 	(footprint "PCM_kikit:Tab"
 		(layer "F.Cu")
-		(at 131.4 34.19 -90)
+		(at 131.4 35 -90)
 		(descr "A symbol representing annotation for tab placement")
 		(property "Reference" "REF**"
@@
 		(descr "A symbol representing annotation for tab placement")
 		(property "Reference" "REF**"
-			(at -0.25 -2 360)
+			(at -0.25 -2 0)
 			(layer "F.SilkS")
 			(hide yes)
@@
 		)
 		(property "Value" "Tab"
-			(at -3 -1 360)
+			(at -3 -1 0)
 			(layer "Dwgs.User")
 			(effects
@@
 		)
 		(property "Footprint" "PCM_kikit:Tab"
-			(at 0 0 360)
+			(at 0 0 0)
 			(layer "F.Fab")
 			(hide yes)
@@
 		)
 		(property "Datasheet" ""
-			(at 0 0 360)
+			(at 0 0 0)
 			(layer "F.Fab")
 			(hide yes)
@@
 		)
 		(property "Description" ""
-			(at 0 0 360)
+			(at 0 0 0)
 			(layer "F.Fab")
 			(hide yes)
@@
 			(layer "Dwgs.User")
 		)
-		(fp_text user "KIKIT: width: 4mm"
+		(fp_text user "KIKIT: width: 3mm"
 			(at -5.5 0 90)
 			(layer "Dwgs.User")
@@
 			(layer "Dwgs.User")
 		)
-		(fp_text user "KIKIT: width: 4mm"
+		(fp_text user "KIKIT: width: 3mm"
 			(at -5.5 0 90)
 			(layer "Dwgs.User")
@@
 		(layer "F.Fab")
 	)
-	(gr_text "DC-DC converter\nVin: 13-60V\nVout: 12V\nMax Out: 3A"
-		(at 114.31 37.49 180)
+	(gr_text "DC-DC Converter\nInput: 13-60V\nOutput: 12V\nMax Output: 3A\n"
+		(at 116.79 38.73 180)
+		(layer "B.SilkS")
+		(effects
+			(font
+				(size 1.5 1.5)
+				(thickness 0.2)
+			)
+			(justify left bottom mirror)
+		)
+	)
+	(gr_text "Gnd"
+		(at 103.17 42.5 180)
 		(layer "B.SilkS")
 		(effects
@@
 				(thickness 0.15)
 			)
-			(justify left bottom mirror)
+			(justify mirror)
 		)
 	)
@@
 	)
 	(gr_text "12V"
-		(at 110.8 36.2 180)
+		(at 110.73 42.5 180)
+		(layer "B.SilkS")
+		(effects
+			(font
+				(size 1 1)
+				(thickness 0.15)
+			)
+			(justify mirror)
+		)
+	)
+	(gr_text "12V"
+		(at 110.78 42.5 180)
 		(layer "F.SilkS")
 		(effects
@@
 	)
 	(gr_text "Gnd"
-		(at 103.2 36 180)
+		(at 103.2 42.5 180)
 		(layer "F.SilkS")
 		(effects
@@
 	)
 	(gr_text "${TAG}"
-		(at 99.6 64.71 180)
+		(at 136.43 46.03 -90)
 		(layer "F.SilkS")
 		(effects
@@
 	(zone
 		(net 7)
-		(net_name "Net-(J1-Pin_2)")
+		(net_name "/VCC_Pre_Fuse")
 		(layer "F.Cu")
 		(hatch edge 0.508)
@@
 	(zone
 		(net 8)
-		(net_name "Net-(J2-Pin_1)")
+		(net_name "/12V_Fused")
 		(layer "F.Cu")
 		(hatch edge 0.508)
