File: battery-dc-dc/battery-dc-dc.kicad_sch (KiCad schematic)
At the start: 24 parts, among them J1 Conn_01x02, J2 Conn_01x01, J3 Conn_01x01, U1 LMR16030P

Commit message: 0.4.0 release
Parts:
- J2, J3: now left out of the parts list
Changed lines of the file:
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@@
 		(unit 1)
 		(exclude_from_sim no)
-		(in_bom yes)
+		(in_bom no)
 		(on_board yes)
 		(dnp no)
@@
 		(unit 1)
 		(exclude_from_sim no)
-		(in_bom yes)
+		(in_bom no)
 		(on_board yes)
 		(dnp no)
